File: KiCad/Spark-AE.kicad_sch (KiCad schematic)
At the start: 1 part

Commit message: Roughing out the basic edges and control layout.
Parts:
- removed A1: Electrosmith_Daisy_Seed_Rev4, Module:Electrosmith_Daisy_Seed, symbol MCU_Module:Electrosmith_Daisy_Seed_Rev4
Changed lines of the file:
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@@
 	(generator_version "9.0")
 	(paper "A4")
-	(symbol
-		(lib_id "MCU_Module:Electrosmith_Daisy_Seed_Rev4")
-		(at 88.9 74.93 0)
-		(unit 1)
-		(exclude_from_sim no)
-		(in_bom yes)
-		(on_board yes)
-		(dnp no)
-		(fields_autoplaced yes)
-		(property "Reference" "A1"
-			(at 93.5833 110.49 0)
-			(effects
-				(font
-					(size 1.27 1.27)
-				)
-				(justify left)
-			)
-		)
-		(property "Value" "Electrosmith_Daisy_Seed_Rev4"
-			(at 93.5833 113.03 0)
-			(effects
-				(font
-					(size 1.27 1.27)
-				)
-				(justify left)
-			)
-		)
-		(property "Footprint" "Module:Electrosmith_Daisy_Seed"
-			(at 107.95 110.49 0)
-			(effects
-				(font
-					(size 1.27 1.27)
-				)
-				(hide yes)
-			)
-		)
-		(property "Datasheet" "https://static1.squarespace.com/static/58d03fdc1b10e3bf442567b8/t/6227e6236f02fb68d1577146/1646781988478/Daisy_Seed_datasheet_v1.0.3.pdf"
-			(at 166.37 113.03 0)
-			(effects
-				(font
-					(size 1.27 1.27)
-				)
-				(hide yes)
-			)
-		)
-		(property "Description" "Daisy is an embedded platform for music."
-			(at 88.9 74.93 0)
-			(effects
-				(font
-					(size 1.27 1.27)
-				)
-				(hide yes)
-			)
-		)
-		(pin "19"
-		)
-		(pin "22"
-		)
-		(pin "23"
-		)
-		(pin "24"
-		)
-		(pin "25"
-		)
-		(pin "26"
-		)
-		(pin "27"
-		)
-		(pin "28"
-		)
-		(pin "29"
-		)
-		(pin "30"
-		)
-		(pin "31"
-		)
-		(pin "32"
-		)
-		(pin "33"
-		)
-		(pin "34"
-		)
-		(pin "35"
-		)
-		(pin "39"
-		)
-		(pin "40"
-		)
-		(pin "38"
-		)
-		(pin "21"
-		)
-		(pin "16"
-		)
-		(pin "17"
-		)
-		(pin "18"
-		)
-		(pin "20"
-		)
-		(pin "1"
-		)
-		(pin "36"
-		)
-		(pin "37"
-		)
-		(pin "14"
-		)
-		(pin "15"
-		)
-		(pin "12"
-		)
-		(pin "13"
-		)
-		(pin "8"
-		)
-		(pin "9"
-		)
-		(pin "10"
-		)
-		(pin "11"
-		)
-		(pin "5"
-		)
-		(pin "4"
-		)
-		(pin "3"
-		)
-		(pin "2"
-		)
-		(pin "6"
-		)
-		(pin "7"
-		)
-		(instances
-			(project ""
-				(path "/6d565a13-335b-43b0-9923-7e064a666c57"
-					(reference "A1")
-					(unit 1)
-				)
-			)
-		)
-	)
 	(sheet_instances
 		(path "/"

Commit message: removed led holes in favor of transparent pots
Other:
- company: (none) -> Copyright © 2026 clectric.diy Licensed under CERN-OHL-S v2
- title: (none) -> Spark-AE
Changed lines of the file:
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@@
 	(generator_version "9.0")
 	(paper "A4")
+	(title_block
+		(title "Spark-AE")
+		(date "2026-01-14")
+		(company "Copyright © 2026 clectric.diy Licensed under CERN-OHL-S v2")
+		(comment 1 "Charles H. Leggett")
+	)
 	(sheet_instances
 		(path "/"
