File: KiCad/Spark-AE-Lower/Spark-AE-Lower.kicad_sch (KiCad schematic)
At the start: 0 parts

Commit message: filled in title blocks
Other:
- company: (none) -> Copyright © 2025 clectric.diy Licensed under CERN-OHL-S v2
- title: (none) -> Spark-AE-Lower
Changed lines of the file:
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@@
 	(generator_version "9.0")
 	(paper "A4")
+	(title_block
+		(title "Spark-AE-Lower")
+		(date "2026-01-14")
+		(rev "0.1")
+		(company "Copyright © 2025 clectric.diy Licensed under CERN-OHL-S v2")
+		(comment 1 "Charles H. Leggett")
+	)
 	(sheet_instances
 		(path "/"
