File: KiCad/Spark-AE/Spark-AE-Panel/Spark-AE-Panel.kicad_sch (KiCad schematic)
At the start: 0 parts

Commit message: pcb layout complete. ready for final pre-fab confirmation.
Parts:
- added C31: 10uF, Capacitor_SMD:C_0603_1608Metric, symbol Device:C
- added C32: 100nF, Capacitor_SMD:C_0603_1608Metric, symbol Device:C
- added R57, R58, R59, R60, R61: 47K, Resistor_SMD:R_0603_1608Metric, symbol Device:R_US
- added U7: Connector_Micro_SD_Card_Yamaichi_PJS008U-3000-0, clectric-diy:PJS008U-3000-0, symbol clectric-diy:Connector_Micro_SD_Card_Yamaichi_PJS008U-3000-0
Connections:
- new net +3.3V: C31.1, C32.1, R57.1, R58.1, R59.1, R60.1, R61.1, U7.P$4 (4_VDD)
- new net GND: C31.2, C32.2, U7.P$10 (HOUSING_2), U7.P$6 (6_VSS/GND), U7.P$9 (HOUSING_1)
- new net SD_CK: U7.P$5 (5_CLK)
- new net SD_CMD: R59.2, U7.P$3 (3_CMD/DI)
- new net SD_D0: R58.2, U7.P$7 (7_DAT0/D0)
- new net SD_D1: R57.2, U7.P$8 (8_DAT1/X)
- new net SD_D2: R61.2, U7.P$1 (1_DAT2/X)
- new net SD_D3: R60.2, U7.P$2 (2_CD/DAT3/CS)
